File: ESP32C3-Biceps_Shoulder/KiCad_resolution/KiCad_resolution.kicad_sch (KiCad schematic)
At the start: 2 parts, among them U1 ESP32-C3-DevKitM-1

Commit message: Commit 5 (Added PCB file , added BNO_055 library of view)
Parts:
- BNO_055_9DOF2: footprint (none) -> BNO_055:Без назви
Connections:
- no-connect marks 0 -> 17
Changed lines of the file:
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@@
 	(generator_version "10.0")
 	(paper "A4")
+	(no_connect
+		(at 118.11 101.6)
+	)
+	(no_connect
+		(at 130.81 101.6)
+	)
+	(no_connect
+		(at 120.65 132.08)
+	)
+	(no_connect
+		(at 128.27 101.6)
+	)
+	(no_connect
+		(at 125.73 101.6)
+	)
+	(no_connect
+		(at 137.16 85.09)
+	)
+	(no_connect
+		(at 148.59 85.09)
+	)
+	(no_connect
+		(at 144.78 85.09)
+	)
+	(no_connect
+		(at 130.81 132.08)
+	)
+	(no_connect
+		(at 133.35 132.08)
+	)
+	(no_connect
+		(at 138.43 132.08)
+	)
+	(no_connect
+		(at 120.65 101.6)
+	)
+	(no_connect
+		(at 123.19 101.6)
+	)
+	(no_connect
+		(at 138.43 101.6)
+	)
+	(no_connect
+		(at 118.11 132.08)
+	)
+	(no_connect
+		(at 135.89 101.6)
+	)
+	(no_connect
+		(at 133.35 101.6)
+	)
 	(wire
 		(pts
@@
 			)
 		)
-		(property "Footprint" ""
+		(property "Footprint" "BNO_055:Без назви"
 			(at 129.54 78.74 0)
 			(hide yes)
